Commit message: Tower link and joint created - still not appearing on rviz

File: agrob_description/urdf/agrob.urdf.xacro (robot description, xacro)
@@ -1,11 +1,37 @@
 <?xml version="1.0"?>
 <robot xmlns:xacro="http://www.ros.org/wiki/xacro" name="agrob">
-    <xacro:include filename="$(find husky_description)/urdf/husky.urdf.xacro" />
-    <xacro:include filename="$(find hector_sensors_description)/urdf/vlp16.urdf.xacro" />
+    <!--<xacro:include filename="$(find husky_description)/urdf/husky.urdf.xacro" />-->
+    <!-- <xacro:include filename="$(find hector_sensors_description)/urdf/vlp16.urdf.xacro" /> -->
     <xacro:macro name="agrob" params="prefix">
         <!-- vehicle model -->
-        <xacro:husky />
+        <!--<xacro:husky />-->
         <!-- velodyne-16 model -->
-        <xacro:vlp16_model />
+        <!--<xacro:vlp16_model /> -->
+      <link name="tower_link">
+        <visual>
+          <origin xyz="0 0 0" rpy="0 0 0" />
+          <geometry>
+            <box size="0.3 0.3 0.8" />
+          </geometry>
+        </visual>
+      </link>
+      <link name="tower_link_2">
+        <visual>
+          <origin xyz="0 0 0" rpy="0 0 0" />
+          <geometry>
+            <box size="0.3 0.3 0.8" />
+          </geometry>
+        </visual>
+      </link>
+      <joint name="tower_link-tower_link_2" type="fixed">
+        <parent link="tower_link"/>
+        <child link="tower_link_2"/>
+        <origin xyz="-0.15 0 0" rpy="0 0 0" />
+      </joint>
+      <joint name="top_plate_front_link_tower_link" type="fixed">
+        <parent link="top_plate_front_link"/>
+        <child link="tower_link"/>
+        <origin xyz="-0.15 0 0" rpy="0 0 0" />
+      </joint>
     </xacro:macro>
 </robot>

Commit message: Creating links and joints in the agrob xacro ...

File: agrob_description/urdf/agrob.urdf.xacro (robot description, xacro)
@@ -1,37 +1,28 @@
 <?xml version="1.0"?>
 <robot xmlns:xacro="http://www.ros.org/wiki/xacro" name="agrob">
-    <!--<xacro:include filename="$(find husky_description)/urdf/husky.urdf.xacro" />-->
-    <!-- <xacro:include filename="$(find hector_sensors_description)/urdf/vlp16.urdf.xacro" /> -->
+    <xacro:include filename="$(find husky_description)/urdf/husky.urdf.xacro" />
+     <xacro:include filename="$(find hector_sensors_description)/urdf/vlp16.urdf.xacro" />
     <xacro:macro name="agrob" params="prefix">
         <!-- vehicle model -->
-        <!--<xacro:husky />-->
+<!--        <xacro:husky />-->
         <!-- velodyne-16 model -->
-        <!--<xacro:vlp16_model /> -->
-      <link name="tower_link">
-        <visual>
-          <origin xyz="0 0 0" rpy="0 0 0" />
-          <geometry>
-            <box size="0.3 0.3 0.8" />
-          </geometry>
-        </visual>
-      </link>
-      <link name="tower_link_2">
-        <visual>
-          <origin xyz="0 0 0" rpy="0 0 0" />
-          <geometry>
-            <box size="0.3 0.3 0.8" />
-          </geometry>
-        </visual>
-      </link>
-      <joint name="tower_link-tower_link_2" type="fixed">
-        <parent link="tower_link"/>
-        <child link="tower_link_2"/>
-        <origin xyz="-0.15 0 0" rpy="0 0 0" />
-      </joint>
-      <joint name="top_plate_front_link_tower_link" type="fixed">
-        <parent link="top_plate_front_link"/>
-        <child link="tower_link"/>
-        <origin xyz="-0.15 0 0" rpy="0 0 0" />
-      </joint>
+        <xacro:vlp16_model name="vlp16" parent="tower_link">
+            <origin xyz="0 0 0" rpy="0 0 0"/>
+        </xacro:vlp16_model>
+        <link name="tower_link">
+          <visual>
+            <origin xyz="0 0 0" rpy="0 0 0" />
+            <geometry>
+              <box size="0.3 0.3 0.8" />
+            </geometry>
+          </visual>
+        </link>
+        <joint name="top_plate_front_link_tower_link" type="fixed">
+          <parent link="top_plate_front_link"/>
+          <child link="tower_link"/>
+          <origin xyz="-0.15 0 0" rpy="0 0 0" />
+        </joint>
     </xacro:macro>
+    <!-- Call the xacro macro-->
+    <xacro:agrob prefix=""/>
 </robot>

Commit message: Color added to tower_link

File: agrob_description/urdf/agrob.urdf.xacro (robot description, xacro)
@@ -5,4 +5,7 @@
      <xacro:include filename="$(find hector_sensors_description)/urdf/vlp16.urdf.xacro" />
     <xacro:macro name="agrob" params="prefix">
+    <material name="tower_color">
+        <color rgba="0 0 0.8 1"/>
+    </material>
         <!-- vehicle model -->
 <!--        <xacro:husky />-->
@@ -16,4 +19,5 @@
             <geometry>
               <box size="0.3 0.3 0.8" />
+              <material name="tower_color" />
             </geometry>
           </visual>

Commit message: Solving inertia tensors problem

File: agrob_description/urdf/agrob.urdf.xacro (robot description, xacro)
@@ -6,5 +6,5 @@
     <xacro:macro name="agrob" params="prefix">
     <material name="tower_color">
-        <color rgba="0 0 0.8 1"/>
+        <color rgba="1 0 0.8 1"/>
     </material>
         <!-- vehicle model -->
@@ -19,6 +19,6 @@
             <geometry>
               <box size="0.3 0.3 0.8" />
-              <material name="tower_color" />
             </geometry>
+            <material name="tower_color" />
           </visual>
         </link>

Commit message: tower designed using solidworks & zed urdf added

File: agrob_description/urdf/agrob.urdf.xacro (robot description, xacro)
@@ -3,29 +3,73 @@
     <xacro:include filename="$(find hector_xacro_tools)/urdf/inertia_tensors.urdf.xacro"/>
     <xacro:include filename="$(find husky_description)/urdf/husky.urdf.xacro" />
-     <xacro:include filename="$(find hector_sensors_description)/urdf/vlp16.urdf.xacro" />
+    <xacro:include filename="$(find hector_sensors_description)/urdf/vlp16.urdf.xacro" />
     <xacro:macro name="agrob" params="prefix">
-    <material name="tower_color">
-        <color rgba="1 0 0.8 1"/>
+    <material name="towercolor">
+        <color rgba="0.86 0.86 0.86 1"/>
     </material>
-        <!-- vehicle model -->
-<!--        <xacro:husky />-->
         <!-- velodyne-16 model -->
         <xacro:vlp16_model name="vlp16" parent="tower_link">
-            <origin xyz="0 0 0" rpy="0 0 0"/>
+            <origin xyz="0 0.6327 0" rpy="-1.57 0 0"/>
         </xacro:vlp16_model>
+        <!-- zed camera model -->
+        <link name="zed_camera_center">
+            <visual>
+                <origin xyz="0 0 0" rpy="0 0 0"/>
+                <geometry>
+                    <mesh filename="package://agrob_description/meshes/ZED.stl" />
+                </geometry>
+                <material name="light_grey">
+                    <color rgba="0.8 0.8 0.8 0.8"/>
+                </material>
+            </visual>
+        </link>
+        <!-- tower model -->
         <link name="tower_link">
           <visual>
             <origin xyz="0 0 0" rpy="0 0 0" />
             <geometry>
-              <box size="0.3 0.3 0.8" />
+              <mesh filename="package://agrob_description/meshes/agrob_tower.STL" />
             </geometry>
-            <material name="tower_color" />
+            <material name="towercolor" />
           </visual>
         </link>
+        <!-- base to tower joint -->
         <joint name="top_plate_front_link_tower_link" type="fixed">
           <parent link="top_plate_front_link"/>
           <child link="tower_link"/>
-          <origin xyz="-0.15 0 0" rpy="0 0 0" />
+          <origin xyz="-0.14 0 0" rpy="1.57 0 0" />
         </joint>
+        <!-- tower to ZED camera center joint -->
+        <joint name="tower_link_zed_camera_center" type="fixed">
+          <parent link="tower_link"/>
+          <child link="zed_camera_center"/>
+          <origin xyz="0.05 0.580 0" rpy="-1.57 0 0" />
+        </joint>
+        <!-- Left ZED Camera -->
+        <joint name="zed_left_camera_joint" type="fixed">
+          <parent link="zed_camera_center"/>
+          <child link="zed_left_camera_frame"/>
+          <origin xyz="0 0.06 0" rpy="0 0 0" />
+        </joint>
+        <link name="zed_left_camera_frame" />
+        <joint name="zed_left_camera_optical_joint" type="fixed">
+          <origin xyz="0 0 0" rpy="-1.57079632679 0.0 -1.57079632679"/>
+          <parent link="zed_left_camera_frame"/>
+          <child link="zed_left_camera_optical_frame"/>
+        </joint>
+        <link name="zed_left_camera_optical_frame"/>
+        <!-- Right ZED Camera -->
+        <joint name="zed_right_camera_joint" type="fixed">
+          <parent link="zed_camera_center"/>
+          <child link="zed_right_camera_frame"/>
+          <origin xyz="0 -0.06 0" rpy="0 0 0" />
+        </joint>
+        <link name="zed_right_camera_frame" />
+        <joint name="zed_right_camera_optical_joint" type="fixed">
+          <origin xyz="0 0 0" rpy="-1.57079632679 0.0 -1.57079632679"/>
+          <parent link="zed_right_camera_frame"/>
+          <child link="zed_right_camera_optical_frame"/>
+        </joint>
+        <link name="zed_right_camera_optical_frame"/>
     </xacro:macro>
     <!-- Call the xacro macro-->

Commit message: #157 temporary fix in the agrob xacro for fixing the problem in the vlp16_frame / velodyne links.

File: agrob_description/urdf/agrob.urdf.xacro (robot description, xacro)
@@ -8,4 +8,16 @@
         <color rgba="0.86 0.86 0.86 1"/>
     </material>
+        <!-- ###################################################### -->
+        <!--To replace the need to add this in the launch file-->
+        <!--<node pkg="tf" type="static_transform_publisher" name="vlp16_to_velodyne" args="0 0 0 0 0 0 1 /vlp16_frame /velodyne 10" />-->
+        <link name="tower_link">
+        </link>
+        <joint name="vlp16_frame_to_velodyne" type="fixed">
+          <parent link="vlp16_frame"/>
+          <child link="velodyne"/>
+          <origin xyz="0 0 0" rpy="0 0 1" />
+        </joint>
+        <!--This must be removed once the bags have the correct velodyne link-->
+        <!-- ###################################################### -->
         <!-- velodyne-16 model -->
         <xacro:vlp16_model name="vlp16" parent="tower_link">

Commit message: #157 fixing the fix ...

File: agrob_description/urdf/agrob.urdf.xacro (robot description, xacro)
@@ -11,5 +11,5 @@
         <!--To replace the need to add this in the launch file-->
         <!--<node pkg="tf" type="static_transform_publisher" name="vlp16_to_velodyne" args="0 0 0 0 0 0 1 /vlp16_frame /velodyne 10" />-->
-        <link name="tower_link">
+        <link name="velodyne">
         </link>
         <joint name="vlp16_frame_to_velodyne" type="fixed">
