Commit message: #199 Fixing velodyne position in agrob xacro

File: agrob_calibration/urdf/initial_estimate.urdf.xacro (robot description, xacro)
@@ -16,5 +16,5 @@
           <parent link="vlp16_frame"/>
           <child link="velodyne"/>
-          <origin xyz="0 0 0" rpy="0 0 1" />
+          <origin xyz="0 0 0" rpy="0 0 0" />
         </joint>
         <!--This must be removed once the bags have the correct velodyne link-->

Commit message: #199 xacro updated with camera pointing down

File: agrob_calibration/urdf/initial_estimate.urdf.xacro (robot description, xacro)
@@ -56,5 +56,5 @@
           <parent link="tower_link"/>
           <child link="zed_camera_center"/>
-          <origin xyz="0.05 0.580 0" rpy="-1.57 0 0" />
+          <origin xyz="0.05 0.580 0" rpy="-1.57  0 -0.174532925" />
         </joint>
         <!-- Left ZED Camera -->
